File: Ergogen assisted/PCBs/boomerang_left.kicad_pcb (KiCad board)
At the start: 2 copper layers, 151.9 x 128.8 mm, 50 parts

Commit message: fix: PCBs positions
Parts:
- moved REF** 5.43 mm to (122.0, 124.3)
- moved MCU2 0.60 mm to (181.6, 127.2)
Connections:
- net p_switch renamed battery_raw
Routing:
- net RAW: track 91.2 -> 96.6 mm
- net battery_raw: track 29.6 -> 34.2 mm
- net P18: track 85.2 -> 83.9 mm
- net GND: track 105.0 -> 106.0 mm
- net RST: track 32.7 -> 33.5 mm
- net P10: track 157.8 -> 158.5 mm
- net P9: track 153.9 -> 154.7 mm
- net P16: track 149.3 -> 150.0 mm
- net P8: track 165.0 -> 165.7 mm
- net P14: track 107.0 -> 107.7 mm
- net P7: track 149.2 -> 149.9 mm
- net P5: track 120.4 -> 121.1 mm
- net P6: track 131.6 -> 132.3 mm
- net P19: track 61.9 -> 61.2 mm
- net P3: track 56.8 -> 57.3 mm
