File: Ergogen assisted/PCBs/boomerang_right.kicad_pcb (KiCad board)
At the start: 2 copper layers, 151.9 x 128.8 mm, 50 parts

Commit message: fix: PCBs positions
Parts:
- moved REF** 2.00 mm to (282.0, 124.2)
- moved MCU1 0.20 mm to (222.4, 127.0)
Routing:
- net P10: track 219.8 -> 218.5 mm
- net P16: track 214.6 -> 213.3 mm
- net P14: track 151.0 -> 150.0 mm
- net p_switch: track 19.4 -> 18.6 mm
- net GND: track 113.5 -> 114.3 mm
- net P20: track 47.3 -> 47.9 mm
- net P8: track 210.2 -> 210.7 mm
- net P7: track 193.2 -> 193.8 mm
- net P4: track 138.2 -> 138.7 mm
- net P6: track 173.7 -> 174.2 mm
- net P19: track 28.2 -> 28.7 mm
